File: AC t0 DC Convertor/AC t0 DC Convertor.kicad_pcb (KiCad board)
At the start: 2 copper layers, 45 x 40.2 mm, 12 parts, among them J1 Screw_Terminal_01x02, J2 Screw_Terminal_01x02

Commit message: Push transformerless PSU design files and updated AC-DC PCB, ignore KiCad backups
Parts:
- added REF**: OSHW-Logo_5.7x6mm_SilkScreen, Symbol:OSHW-Logo_5.7x6mm_SilkScreen, F.Cu at (86.8, 105.1)
